File: raspberry_pi_pico.kicad_sch (KiCad schematic)
At the start: 70 parts, among them J2 Conn_02x20_Counter_Clockwise, J3 Conn_02x20_Counter_Clockwise, J7 Conn_01x01_Pin, U3 Pico

Commit message: Fixed a number of things
Parts:
- added J4, J6: Conn_01x20_Socket, Connector_PinSocket_2.54mm:PinSocket_1x20_P2.54mm_Vertical, symbol Connector:Conn_01x20_Socket
Connections:
- net GND: now also J4.13 (Pin_13), J4.18 (Pin_18), J4.3 (Pin_3), J4.8 (Pin_8), J6.13 (Pin_13), J6.18 (Pin_18), J6.3 (Pin_3), J6.8 (Pin_8)
- net RST: now also J6.11 (Pin_11)
- net at JP51.1 (A), U3.1 (GPIO0): now also J4.1 (Pin_1)
- net at JP54.1 (A), U3.5 (GPIO3): now also J4.5 (Pin_5)
- net at JP63.1 (A), U3.16 (GPIO12): now also J4.16 (Pin_16)
- net at JP49.2 (B), U3.21 (GPIO16): now also J6.20 (Pin_20)
- net at JP65.1 (A), U3.19 (GPIO14): now also J4.19 (Pin_19)
- net at JP42.2 (B), U3.31 (GPIO26_ADC0): now also J6.10 (Pin_10)
- net at JP58.1 (A), U3.10 (GPIO7): now also J4.10 (Pin_10)
- net at JP59.1 (A), U3.11 (GPIO8): now also J4.11 (Pin_11)
- net at JP60.1 (A), U3.12 (GPIO9): now also J4.12 (Pin_12)
- net at JP61.1 (A), U3.14 (GPIO10): now also J4.14 (Pin_14)
- net at JP62.1 (A), U3.15 (GPIO11): now also J4.15 (Pin_15)
- net at JP64.1 (A), U3.17 (GPIO13): now also J4.17 (Pin_17)
- net at JP52.1 (A), U3.2 (GPIO1): now also J4.2 (Pin_2)
- net at JP66.1 (A), U3.20 (GPIO15): now also J4.20 (Pin_20)
- net at JP48.2 (B), U3.22 (GPIO17): now also J6.19 (Pin_19)
- net at JP47.2 (B), U3.24 (GPIO18): now also J6.17 (Pin_17)
- net at JP46.2 (B), U3.25 (GPIO19): now also J6.16 (Pin_16)
- net at JP45.2 (B), U3.26 (GPIO20): now also J6.15 (Pin_15)
- net at JP44.2 (B), U3.27 (GPIO21): now also J6.14 (Pin_14)
- net at JP43.2 (B), U3.29 (GPIO22): now also J6.12 (Pin_12)
- net at JP41.2 (B), U3.32 (GPIO27_ADC1): now also J6.9 (Pin_9)
- net at JP40.2 (B), U3.34 (GPIO28_ADC2): now also J6.7 (Pin_7)
- net at JP39.2 (B), U3.35 (ADC_VREF): now also J6.6 (Pin_6)
- net at JP38.2 (B), U3.36 (3V3): now also J6.5 (Pin_5)
- net at JP37.2 (B), U3.37 (3V3_EN): now also J6.4 (Pin_4)
- net at JP36.2 (B), U3.39 (VSYS): now also J6.2 (Pin_2)
- net at JP53.1 (A), U3.4 (GPIO2): now also J4.4 (Pin_4)
- net at J7.1 (Pin_1), JP50.1 (A), U3.40 (VBUS): now also J6.1 (Pin_1)
- net at JP55.1 (A), U3.6 (GPIO4): now also J4.6 (Pin_6)
- net at JP56.1 (A), U3.7 (GPIO5): now also J4.7 (Pin_7)
- net at JP57.1 (A), U3.9 (GPIO6): now also J4.9 (Pin_9)
