File: raspberry_pi_pico.kicad_sch (KiCad schematic)
At the start: 72 parts, among them J2 Conn_02x20_Counter_Clockwise, J3 Conn_02x20_Counter_Clockwise, J4 Conn_01x20_Socket, J6 Conn_01x20_Socket, J7 Conn_01x01_Pin, U3 Pico

Commit message: Added DAC
Parts:
- removed J6: Conn_01x20_Socket, Connector_PinSocket_2.54mm:PinSocket_1x20_P2.54mm_Vertical, symbol Connector:Conn_01x20_Socket
- added J10: Conn_01x20_Socket, Intro_to_CAD:PinSocket_1x20_P2.54mm_Vertical-pins21-40, symbol Connector:Conn_01x20_Socket
Connections:
- net GND: now also J10.23 (Pin_18), J10.28 (Pin_13), J10.33 (Pin_8), J10.38 (Pin_3)
- net RST: now also J10.30 (Pin_11)
- net at JP49.2 (B), U3.21 (GPIO16): now also J10.21 (Pin_20)
- net at JP42.2 (B), U3.31 (GPIO26_ADC0): now also J10.31 (Pin_10)
- net at JP48.2 (B), U3.22 (GPIO17): now also J10.22 (Pin_19)
- net at JP47.2 (B), U3.24 (GPIO18): now also J10.24 (Pin_17)
- net at JP46.2 (B), U3.25 (GPIO19): now also J10.25 (Pin_16)
- net at JP45.2 (B), U3.26 (GPIO20): now also J10.26 (Pin_15)
- net at JP44.2 (B), U3.27 (GPIO21): now also J10.27 (Pin_14)
- net at JP43.2 (B), U3.29 (GPIO22): now also J10.29 (Pin_12)
- net at JP41.2 (B), U3.32 (GPIO27_ADC1): now also J10.32 (Pin_9)
- net at JP40.2 (B), U3.34 (GPIO28_ADC2): now also J10.34 (Pin_7)
- net at JP39.2 (B), U3.35 (ADC_VREF): now also J10.35 (Pin_6)
- net at JP38.2 (B), U3.36 (3V3): now also J10.36 (Pin_5)
- net at JP37.2 (B), U3.37 (3V3_EN): now also J10.37 (Pin_4)
- net at JP36.2 (B), U3.39 (VSYS): now also J10.39 (Pin_2)
- net at J7.1 (Pin_1), JP50.1 (A), U3.40 (VBUS): now also J10.40 (Pin_1)
