File: VDDA.kicad_sch (KiCad schematic)
At the start: 30 parts, among them J5 Conn_01x02, Q1 AO3401A, U6 L78M05ABDT-TR

Commit message: Some insurance added to the DAC Amp
Connections:
- net VAH: now reaches C41.1, D2.1, Q1.1 (G), R21.2, R28.1, U6.1 (VIN)
Changed lines of the file:
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@@
 	)
 	(junction
+		(at 102.87 67.31)
+		(diameter 0)
+		(color 0 0 0 0)
+	)
+	(junction
 		(at 161.29 115.57)
 		(diameter 0)
@@
 	(wire
 		(pts
-			(xy 102.87 64.77) (xy 102.87 73.66)
+			(xy 102.87 64.77) (xy 102.87 67.31)
 		)
 		(stroke
@@
 	(wire
 		(pts
+			(xy 102.87 67.31) (xy 102.87 73.66)
+		)
+		(stroke
+			(width 0)
+			(type default)
+		)
+	)
+	(wire
+		(pts
 			(xy 59.69 113.03) (xy 62.23 113.03)
 		)
@@
 					(unit 1)
 				)
+			)
+		)
+	)
+	(symbol
+		(lib_id "power:VDDA")
+		(at 102.87 67.31 270)
+		(unit 1)
+		(exclude_from_sim no)
+		(in_bom yes)
+		(on_board yes)
+		(dnp no)
+		(fields_autoplaced yes)
+		(property "Reference" "#PWR093"
+			(at 99.06 67.31 0)
+			(effects
+				(font
+					(size 1.27 1.27)
+				)
+				(hide yes)
+			)
+		)
+		(property "Value" "VAH"
+			(at 106.68 67.3099 90)
+			(effects
+				(font
+					(size 1.27 1.27)
+				)
+				(justify left)
+			)
+		)
+		(property "Footprint" ""
+			(at 102.87 67.31 0)
+			(effects
+				(font
+					(size 1.27 1.27)
+				)
+				(hide yes)
+			)
+		)
+		(property "Datasheet" ""
+			(at 102.87 67.31 0)
+			(effects
+				(font
+					(size 1.27 1.27)
+				)
+				(hide yes)
+			)
+		)
+		(property "Description" ""
+			(at 102.87 67.31 0)
+			(effects
+				(font
+					(size 1.27 1.27)
+				)
+				(hide yes)
+			)
+		)
+		(pin "1"
+		)
+		(instances
+			(project "Intro-to-CAD-2026"
+				(path "/c12dc015-e6cb-468c-8de4-269c3106de0e/ed314b6d-b133-4548-ae58-2db461511a12"
+					(reference "#PWR093")
+					(unit 1)
+				)
