File: dac.kicad_sch (KiCad schematic)
At the start: 50 parts, among them J9 DAC OUT, Q2 FMMT591, Q3 FMMT491, Q4 FMMT491, Q5 FMMT591, U1 CJC4334H, U9 OPA1612AxD

Commit message: Some insurance added to the DAC Amp
Parts:
- added C61: 100nF, PCM_JLCPCB:C_0805, symbol PCM_JLCPCB-Capacitors:0805,100nF
- added C63: 10uF, PCM_JLCPCB:C_0805, symbol PCM_JLCPCB-Capacitors:0805,10uF,(2)
- added JP3: ~, Jumper:SolderJumper-2_P1.3mm_Open_RoundedPad1.0x1.5mm, symbol Jumper:Jumper_2_Open
- added TP8: V_R, TestPoint:TestPoint_THTPad_D1.5mm_Drill0.7mm, symbol Connector:TestPoint
- added e2, e6, e7: ~, Jumper:SolderJumper-2_P1.3mm_Bridged_RoundedPad1.0x1.5mm, symbol Jumper:Jumper_2_Bridged
Connections:
- net GNDA: now also C61.2, C63.2
- net VDDA: now also JP3.2 (B); no longer C56.2, Q3.3 (C), Q4.3 (C), R39.1, R42.1, R46.1, R53.2, U9.8 (V+)
- net at C53.1, R33.2: now also e7.2 (B); no longer C58.1
- net at C59.1, R40.1, R41.2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: now also TP8.1
- net at C49.1, R22.2: now also e6.1 (A); no longer C57.1
- new net: C58.1, e7.1 (A)
- new net: C57.1, e6.2 (B)
- new net VAH: e2.2 (B)
- new net VAO: C56.2, C61.1, C63.1, JP3.1 (A), Q3.3 (C), Q4.3 (C), R39.1, R42.1, R46.1, R53.2, U9.8 (V+), e2.1 (A)
Other:
- note added: "This wire can be 0.127 mm wide."
- note added: "You will need to move the audio out jack (J9) and the components below it to your part of the board from mine."
- note removed: "I suggest on the third layer down, run a 0.6 mm trace over to the area under your module and make an area there on that layer VDDA. You can look how I did it on my part of the board. You will need to move the audio out jack (J9) and the components below it to your part of the board from mine."
