File: qsd-sdr.kicad_sch (KiCad schematic)
At the start: 51 parts, among them J11 SDR ANT, J12 SDR Out, U5 OPA1612AxD, U7 SN74CBT3253, U8 OPA1612AxD

Commit message: Updated simulations.
Parts:
- added R58, R59, R60, R61: 10Ω, PCM_JLCPCB:R_0402, symbol PCM_JLCPCB-Resistors:0402,10Ω
Connections:
- net at C14.1, C16.1, TP14.1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: now also R60.1; no longer U8.5 (+)
- net at C19.1, C25.1, TP16.1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: now also R59.1; no longer U8.3 (+)
- net at C22.1, C26.1, TP6.1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: now also R61.1; no longer U5.3 (+)
- net at C24.1, C27.1, TP7.1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: now also R58.1; no longer U5.5 (+)
- new net: R61.2, U5.3 (+)
- new net: R58.2, U5.5 (+)
- new net: R59.2, U8.3 (+)
- new net: R60.2, U8.5 (+)
