File: Frohne/Frohne.kicad_sch (KiCad schematic)
At the start: 6 parts

Commit message: Moved my development to Frohne
Other:
- removed sheet Module_Template
- sheet Raspberry_Pi_Pico: file raspberry_pi_pico.kicad_sch -> ../raspberry_pi_pico.kicad_sch
- note added: "Before merging modules, delete the Pico submodule. It is here for reference. It does reference the main Pico schematic, so it will be up to date. Any changes you make to this schematic, you will need to make in the root schematic up a directory."
- note removed: "100 Ohm resistors for Isolation between different users of the I2C."
- note removed: "Open the Module_Template project file in KiCad. Then do File-Save As, and save it as your module project name. Then you need to add a module here like this that points to your Module schematic to this sheet. Be sure to do it with a relative path, not an absolute one."
- company: WWU -> (none)
- title: PCM1808_Sound_Card -> (none)
- moved on the sheet: R15, R23, R24, R25, R26, R27

Commit message: Added DAC
Connections:
- no-connect marks 22 -> 19
Other:
- added sheet CMOS Oscillator (cmos_oscillator.kicad_sch)
- added sheet DAC (dac.kicad_sch)
- note added: "CHanges made to the Pico Module need to be propagated to the main schematic and to the Module Template Schematic before turning students loose to do their modules."
- note removed: "Before merging modules, delete the Pico submodule. It is here for reference. It does reference the main Pico schematic, so it will be up to date. Any changes you make to this schematic, you will need to make in the root schematic up a directory."
