File: Frohne/Frohne.kicad_sch (KiCad schematic)
At the start: 6 parts

Commit message: Tuned length of I and Q.
Other:
- sheet Si5351a ports: added CLK_N, CLK_P; removed CLK0, CLK1
Changed lines of the file:
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@@
 			)
 		)
-		(pin "CLK0" output
+		(pin "CLK_P" output
 			(at 82.55 158.75 0)
 			(effects
@@
 			)
 		)
-		(pin "CLK1" output
+		(pin "CLK_N" output
 			(at 82.55 160.655 0)
 			(effects
