File: Frohne/VDDA.kicad_sch (KiCad schematic)
At the start: 29 parts, among them J5 Conn_01x02, Q1 AO3401A, U6 L78M05ABDT-TR

Commit message: Added DAC
Parts:
- added JP2: ~, Jumper:SolderJumper-2_P1.3mm_Open_RoundedPad1.0x1.5mm, symbol Jumper:Jumper_2_Open
Connections:
- net +4.7: now also JP2.2 (B)
- net at C43.1, D3.2, U6.3 (VOUT): now also JP2.1 (A)
Other:
- moved on the sheet: C17, C2, C35, C36, C37, C40, C41, C42, C43, C5, C55, D1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
