File: Frohne/VDDA.kicad_sch (KiCad schematic)
At the start: 30 parts, among them J5 Conn_01x02, Q1 AO3401A, U6 L78M05ABDT-TR

Commit message: 40 unconnected
Connections:
- net +4.7 is gone; now on net +4.7V: D3.1, JP2.2 (B)
Changed lines of the file:
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@@
 			)
 		)
-		(property "Value" "+4.7"
+		(property "Value" "+4.7V"
 			(at 187.96 73.6599 90)
 			(effects
