File: Frohne/pcm1808.kicad_sch (KiCad schematic)
At the start: 26 parts, among them J1 ADC IN, U2 PCM1808PWR, X2 YC24.576MUBCE2O

Commit message: Added DAC
Parts:
- removed JP17: Jumper_2_Bridged, Jumper:SolderJumper-2_P1.3mm_Bridged2Bar_RoundedPad1.0x1.5mm, symbol Jumper:Jumper_2_Bridged
- removed R14: 100Ω, PCM_JLCPCB:R_0805, symbol PCM_JLCPCB-Resistors:0805,100Ω
- removed R19, R22: 33Ω, PCM_JLCPCB:R_0805, symbol PCM_JLCPCB-Resistors:0805,33Ω
- removed X2: YC24.576MUBCE2O, Oscillator:Oscillator_SMD_Abracon_ASE-4Pin_3.2x2.5mm, symbol Oscillator:ASE-xxxMHz
- added C51: 100nF, PCM_JLCPCB:C_0805, symbol PCM_JLCPCB-Capacitors:0805,100nF
- added R14: 10Ω, PCM_JLCPCB:R_0603, symbol PCM_JLCPCB-Resistors:0603,10Ω
- added e4: Groundloop_Insurance, Jumper:SolderJumper-2_P1.3mm_Bridged_RoundedPad1.0x1.5mm, symbol Jumper:Jumper_2_Bridged
Connections:
- net GND: now also C51.1, R14.2, e4.1 (A)
- net at J1.S: now also C51.2, R14.1, e4.2 (B)
- net SKCI: now reaches U2.6 (SCKI)
Other:
- note removed: "Jumper and resistor for ground loop mediation"
