File: Frohne/Frohne.kicad_pcb (KiCad board)
At the start: 4 copper layers, 100 x 100 mm, 215 parts, among them J1 ADC IN, J10 Conn_01x20_Socket, J11 SDR ANT, J12 SDR Out, J2 Conn_02x20_Counter_Clockwise, J3 Conn_02x20_Counter_Clockwise, J4 Conn_01x20_Socket, J5 Conn_01x02, J7 Conn_01x01_Pin, J8 BNC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

Commit message: 40 unconnected
Parts:
- moved TP5 36.9 mm to (123.7, 97.2)
- moved TP3 14.7 mm to (135.0, 100.8)
- moved J8 8.04 mm to (144.7, 101.4)
Connections:
- D3 pad 1: +4.7 -> +4.7V
- JP2 pad 2: +4.7 -> +4.7V
Routing:
- net Net-(Q1-G): track 4.93 -> 107.1 mm, vias 0 -> 2
- net Net-(Q1-D): track 3.22 -> 93.5 mm, vias 0 -> 2
- net GND: track 24.0 -> 75.3 mm, vias 18 -> 59
- net +4.7V: track 0.00 -> 40.4 mm, vias 0 -> 2
- net /Raspberry_Pi_Pico/RST: track 0.00 -> 18.8 mm
- net /Raspberry_Pi_Pico/GPIO12: track 0.00 -> 13.5 mm
- net /Raspberry_Pi_Pico/GPIO13: track 0.00 -> 12.5 mm
- net /Si5351a/CLK2: track 16.3 -> 24.8 mm
- net Net-(C4-Pad2): track 7.02 -> 13.4 mm
- net Net-(JP2-A): track 0.00 -> 6.33 mm
- net +3.3V: track 18.0 -> 23.6 mm, vias 5 -> 12
- net Net-(U4-CLK0): track 3.10 -> 5.38 mm
- net Net-(U1-VDD): track 8.11 -> 6.96 mm
