File: Frohne/Frohne.kicad_pcb (KiCad board)
At the start: 4 copper layers, 100 x 100 mm, 214 parts, among them J1 ADC IN, J10 Conn_01x20_Socket, J11 SDR ANT, J12 SDR Out, J2 Conn_02x20_Counter_Clockwise, J3 Conn_02x20_Counter_Clockwise, J4 Conn_01x20_Socket, J5 Conn_01x02, J8 BNC, J9 DAC OUT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

Commit message: 410 warnings
Parts:
- added J7: Conn_01x01_Pin, Connector_PinHeader_2.54mm:PinHeader_1x01_P2.54mm_Vertical, F.Cu at (147.8, 33.3)
- J12: value SDR Out -> SDR OUT
- S1: value Tactile Button, 160gf -> RST
Routing:
- net Net-(J10-Pin_1): track 3.09 -> 15.5 mm, vias 0 -> 1
- net GND: track 144.9 -> 147.9 mm, vias 69 -> 70
- net +3.3V: track 26.1 -> 28.7 mm, vias 12 -> 14
